File: hardware/Buck 100V.sch (EAGLE design)
At the start: 0 parts

Commit message: More progress on schematic.
Parts:
- added C1, C4: 4.7uF 100V, rcl:C-USC0603
- added C2: 15uF 100V, rcl:CPOL-USE2,5-6E
- added C3: 0.05uF, rcl:C-USC0603
- added C5: 1000pF, rcl:C-USC0603
- added C6: (no value), rcl:C-USC2220K
- added L1: 33.0UH, LED-drivers:ASPI-0612FS
- added M2: SI5435BDC, LED-drivers:SI5435BDC
- added Q2: FMMT723, zetex:FMMT723
- added R1: 16.9K, rcl:R-US_R0402
- added R2: 47k, rcl:R-US_R0402
- added R3: 28.7k, rcl:R-US_R0402
- added R4: 11K, rcl:R-US_R0402
- added R5, R6, R7: 200K, rcl:R-US_R0402
- added RIS_PTH: (no value), rcl:R-US_0204/7
- added RIS_SMD: (no value), rcl:R-US_R2512
- added RT1: NCP18WF104J03RB, rcl:R-US_R0402
- added U1: LT3756EMSE, LED-drivers:LT3756EMSE
Connections:
- new net /OPEN_LED: U1./OPENLED_SYNC
- new net CTRL: R1.1, RT1.2, U1.CTRL
- new net GND: C1.2, C2.-, C3.2, C4.2, C5.2, R3.1, R4.1, RT1.1, U1.GND
- new net LED_A: M2.D
- new net LED_C: C6.1, L1.2, R7.2
- new net N$1: C3.1, U1.SS
- new net N$2: C4.1, U1.INTVCC
- new net N$3: R2.2, U1.VC
- new net N$4: C5.1, R2.1
- new net N$5: R3.2, U1.RT
- new net N$6: Q2.C, R4.2, U1.FB
- new net N$7: Q2.E, R5.1
- new net N$8: Q2.B, R6.1, R7.1
- new net N$9: M2.S, RIS_PTH.1, RIS_SMD.1
- new net PWM: U1.PWM
- new net SHDN: U1./SHDN
- new net V+: C1.1, C2.+, C6.2, R5.2, R6.2, RIS_PTH.2, RIS_SMD.2, U1.VIN
- new net VREF: R1.2, U1.VREF
