File: hardware/Buck 100V.sch (EAGLE design)
At the start: 31 parts, among them M1 SI3430DV, M2 SI5435BDC, Q1 FMMT625, Q2 FMMT723, U1 LT3756EMSE

Commit message: Add board created from schematic. No placement done yet.
Parts:
- C1: device rcl:C-USC0805 -> rcl:C-USC2220K
- C4: value 4.7uF 100V -> 4.7uF 16V
Changed lines of the file:
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@@
 <grid distance="0.1" unitdist="inch" unit="inch" style="lines" multiple="1" display="no" altdistance="0.01" altunitdist="inch" altunit="inch"/>
 <layers>
-<layer number="1" name="Top" color="4" fill="1" visible="no" active="no"/>
-<layer number="16" name="Bottom" color="1" fill="1" visible="no" active="no"/>
-<layer number="17" name="Pads" color="2" fill="1" visible="no" active="no"/>
-<layer number="18" name="Vias" color="2" fill="1" visible="no" active="no"/>
-<layer number="19" name="Unrouted" color="6" fill="1" visible="no" active="no"/>
-<layer number="20" name="Dimension" color="15" fill="1" visible="no" active="no"/>
-<layer number="21" name="tPlace" color="7" fill="1" visible="no" active="no"/>
-<layer number="22" name="bPlace" color="7" fill="1" visible="no" active="no"/>
-<layer number="23" name="tOrigins" color="15" fill="1" visible="no" active="no"/>
-<layer number="24" name="bOrigins" color="15" fill="1" visible="no" active="no"/>
-<layer number="25" name="tNames" color="7" fill="1" visible="no" active="no"/>
-<layer number="26" name="bNames" color="7" fill="1" visible="no" active="no"/>
-<layer number="27" name="tValues" color="7" fill="1" visible="no" active="no"/>
-<layer number="28" name="bValues" color="7" fill="1" visible="no" active="no"/>
+<layer number="1" name="Top" color="4" fill="1" visible="yes" active="no"/>
+<layer number="16" name="Bottom" color="1" fill="1" visible="yes" active="no"/>
+<layer number="17" name="Pads" color="2" fill="1" visible="yes" active="no"/>
+<layer number="18" name="Vias" color="2" fill="1" visible="yes" active="no"/>
+<layer number="19" name="Unrouted" color="6" fill="1" visible="yes" active="no"/>
+<layer number="20" name="Dimension" color="15" fill="1" visible="yes" active="no"/>
+<layer number="21" name="tPlace" color="7" fill="1" visible="yes" active="no"/>
+<layer number="22" name="bPlace" color="7" fill="1" visible="yes" active="no"/>
+<layer number="23" name="tOrigins" color="15" fill="1" visible="yes" active="no"/>
+<layer number="24" name="bOrigins" color="15" fill="1" visible="yes" active="no"/>
+<layer number="25" name="tNames" color="7" fill="1" visible="yes" active="no"/>
+<layer number="26" name="bNames" color="7" fill="1" visible="yes" active="no"/>
+<layer number="27" name="tValues" color="7" fill="1" visible="yes" active="no"/>
+<layer number="28" name="bValues" color="7" fill="1" visible="yes" active="no"/>
 <layer number="29" name="tStop" color="7" fill="3" visible="no" active="no"/>
 <layer number="30" name="bStop" color="7" fill="6" visible="no" active="no"/>
@@
 <layer number="35" name="tGlue" color="7" fill="4" visible="no" active="no"/>
 <layer number="36" name="bGlue" color="7" fill="5" visible="no" active="no"/>
-<layer number="37" name="tTest" color="7" fill="1" visible="no" active="no"/>
-<layer number="38" name="bTest" color="7" fill="1" visible="no" active="no"/>
+<layer number="37" name="tTest" color="7" fill="1" visible="yes" active="no"/>
+<layer number="38" name="bTest" color="7" fill="1" visible="yes" active="no"/>
 <layer number="39" name="tKeepout" color="4" fill="11" visible="no" active="no"/>
 <layer number="40" name="bKeepout" color="1" fill="11" visible="no" active="no"/>
@@
 <layer number="44" name="Drills" color="7" fill="1" visible="no" active="no"/>
 <layer number="45" name="Holes" color="7" fill="1" visible="no" active="no"/>
-<layer number="46" name="Milling" color="3" fill="1" visible="no" active="no"/>
-<layer number="47" name="Measures" color="7" fill="1" visible="no" active="no"/>
-<layer number="48" name="Document" color="7" fill="1" visible="no" active="no"/>
-<layer number="49" name="Reference" color="7" fill="1" visible="no" active="no"/>
-<layer number="51" name="tDocu" color="7" fill="1" visible="no" active="no"/>
-<layer number="52" name="bDocu" color="7" fill="1" visible="no" active="no"/>
+<layer number="46" name="Milling" color="3" fill="1" visible="yes" active="no"/>
+<layer number="47" name="Measures" color="7" fill="1" visible="yes" active="no"/>
+<layer number="48" name="Document" color="7" fill="1" visible="yes" active="no"/>
+<layer number="49" name="Reference" color="7" fill="1" visible="yes" active="no"/>
+<layer number="51" name="tDocu" color="7" fill="1" visible="yes" active="no"/>
+<layer number="52" name="bDocu" color="7" fill="1" visible="yes" active="no"/>
 <layer number="91" name="Nets" color="2" fill="1" visible="yes" active="yes"/>
 <layer number="92" name="Busses" color="1" fill="1" visible="yes" active="yes"/>
@@
 <part name="U1" library="LED-drivers" deviceset="LT3756" device="EMSE"/>
 <part name="GND1" library="supply1" deviceset="GND" device=""/>
-<part name="C1" library="rcl" deviceset="C-US" device="C0805" value="4.7uF 100V"/>
+<part name="C1" library="rcl" deviceset="C-US" device="C2220K" value="4.7uF 100V"/>
 <part name="C2" library="rcl" deviceset="CPOL-US" device="E2,5-6E" value="15uF 100V"/>
 <part name="GND2" library="supply1" deviceset="GND" device=""/>
@@
 <part name="GND4" library="supply1" deviceset="GND" device=""/>
 <part name="C3" library="rcl" deviceset="C-US" device="C0805" value="0.047uF"/>
-<part name="C4" library="rcl" deviceset="C-US" device="C0805" value="4.7uF 100V"/>
+<part name="C4" library="rcl" deviceset="C-US" device="C0805" value="4.7uF 16V"/>
 <part name="C5" library="rcl" deviceset="C-US" device="C0805" value="1000pF"/>
 <part name="R2" library="rcl" deviceset="R-US_" device="R0805" value="47k"/>

Commit message: Create kelvin terminated versions of current sense resistors and adjust schematic accordingly. Signals on the buck headers are now more clearly named. The kelvin terminated resistors WILL cause DRC errors on the board due to overlapping vias / pads but these can be safely ignored. Someday perhaps Eagle will get a better way to deal with kelvin termination.
Parts:
- RIS_PTH: device rcl:R-US_0204/7 -> LED-drivers:R-KELVIN0204/7
- RIS_SMD: device rcl:R-US_R2512 -> LED-drivers:R-KELVINR2512
- renumbered R10 to RSENSE
Connections:
- removed net IS: JH.3, M2.S, RIS_PTH.1, RIS_SMD.1, U1.ISN
- new net ISN: JH.3, RIS_PTH.P$1, RIS_SMD.P$1, U1.ISN
- new net ISP: JH.2, RIS_PTH.P$2, RIS_SMD.P$2, U1.ISP
- new net N$7: M2.S, RIS_PTH.1, RIS_SMD.1
- net V+: no longer JH.2, U1.ISP
Other:
- note removed: "R_is"

Commit message: Very rough initial board layout. Can now safely say that the board will be smaller than 2 inches by 3 inches.
Parts:
- renumbered C6 to C_OUT
Connections:
- net N$12 renamed N_BUCK
Changed lines of the file:
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@@
 <part name="JH" library="con-lstb" deviceset="MA06-1" device=""/>
 <part name="JL" library="con-lstb" deviceset="MA08-1" device=""/>
-<part name="C6" library="rcl" deviceset="CPOL-US" device="E2,5-6E" value="15uF 100V"/>
+<part name="C_OUT" library="rcl" deviceset="CPOL-US" device="E2,5-6E" value="15uF 100V"/>
 <part name="RIS_SMD" library="LED-drivers" deviceset="R-KELVIN" device="R2512"/>
 <part name="RIS_PTH" library="LED-drivers" deviceset="R-KELVIN" device="0204/7"/>
@@
 <instance part="JH" gate="1" x="182.88" y="50.8" rot="R180"/>
 <instance part="JL" gate="1" x="182.88" y="22.86" rot="R180"/>
-<instance part="C6" gate="G$1" x="66.04" y="55.88" smashed="yes" rot="R180">
+<instance part="C_OUT" gate="G$1" x="66.04" y="55.88" smashed="yes" rot="R180">
 <attribute name="NAME" x="69.596" y="59.055" size="1.778" layer="95"/>
 <attribute name="VALUE" x="69.596" y="54.229" size="1.778" layer="96"/>
@@
 <wire x1="-58.42" y1="58.42" x2="-58.42" y2="63.5" width="0.1524" layer="91"/>
 <junction x="-58.42" y="63.5"/>
-<pinref part="C6" gate="G$1" pin="-"/>
+<pinref part="C_OUT" gate="G$1" pin="-"/>
 <pinref part="RIS_PTH" gate="G$1" pin="2"/>
 <wire x1="109.22" y1="55.88" x2="109.22" y2="60.96" width="0.1524" layer="91"/>
@@
 <wire x1="66.04" y1="53.34" x2="66.04" y2="43.18" width="0.1524" layer="91"/>
 <junction x="66.04" y="43.18"/>
-<pinref part="C6" gate="G$1" pin="+"/>
+<pinref part="C_OUT" gate="G$1" pin="+"/>
 </segment>
 <segment>
@@
 </segment>
 </net>
-<net name="N$12" class="0">
+<net name="N_BUCK" class="0">
 <segment>
 <pinref part="L1" gate="G$1" pin="1"/>
